Commit message: CHanges

File: description/urdf/five_dof.URDF (robot description, URDF)
Before this commit: robot five_dof, 6 links, 5 joints
Links:
- link base_link: geometry collision mesh filename=file:///home/kaushik/catkin_ws/src/Robotic_Arm_Project/desc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; visual mesh filename=file:///home/kaushik/catkin_ws/src/Robotic_Arm_Project/desc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
- link link1: geometry collision mesh filename=file:///home/kaushik/catkin_ws/src/Robotic_Arm_Project/desc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; visual mesh filename=file:///home/kaushik/catkin_ws/src/Robotic_Arm_Project/desc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
- link link2: geometry collision mesh filename=file:///home/kaushik/catkin_ws/src/Robotic_Arm_Project/desc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; visual mesh filename=file:///home/kaushik/catkin_ws/src/Robotic_Arm_Project/desc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
- link link3: geometry collision mesh filename=file:///home/kaushik/catkin_ws/src/Robotic_Arm_Project/desc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; visual mesh filename=file:///home/kaushik/catkin_ws/src/Robotic_Arm_Project/desc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
- link link4: geometry collision mesh filename=file:///home/kaushik/catkin_ws/src/Robotic_Arm_Project/desc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; visual mesh filename=file:///home/kaushik/catkin_ws/src/Robotic_Arm_Project/desc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
- link link5: geometry collision mesh filename=file:///home/kaushik/catkin_ws/src/Robotic_Arm_Project/desc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; visual mesh filename=file:///home/kaushik/catkin_ws/src/Robotic_Arm_Project/desc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

Commit message: MoveIt Python working

File: description/urdf/five_dof.URDF (robot description, URDF)
Before this commit: robot five_dof, 6 links, 5 joints
Joints:
- joint joint2: limit lower=0.72 upper=2.42 effort=2 velocity=0.03 -> lower=-3.14 upper=3.14 effort=2 velocity=0.03
- joint joint3: limit lower=-2.0 upper=2.0 effort=2 velocity=0.03 -> lower=-3.14 upper=3.14 effort=2 velocity=0.03
- joint joint4: limit lower=-2.5 upper=2.5 effort=2 velocity=0.03 -> lower=-3.14 upper=3.14 effort=2 velocity=0.03
